Commit message: rviz wip

File: mh5_description/urdf/mh5_robot.urdf (robot description, URDF)
Before this commit: robot MH5 Robot, 1 links, 0 joints
Links:
- added link arm_left; visual mesh filename=package://mh5_description/meshes/xl430_with_idle.stl
- added link arm_left_fixed; visual mesh filename=package://mh5_description/meshes/frame03.stl
- added link elbow; visual mesh filename=package://mh5_description/meshes/2xl430_1_idle.stl
- added link hip_left; visual mesh filename=package://mh5_description/meshes/xl430_no_idle.stl
- added link hip_right; visual mesh filename=package://mh5_description/meshes/xl430_no_idle.stl
- added link shoulder_left; visual mesh filename=package://mh5_description/meshes/xl430_no_idle.stl
- added link shoulder_left_frame; visual mesh filename=package://mh5_description/meshes/frame01.stl
- added link shoulder_right; visual mesh filename=package://mh5_description/meshes/xl430_no_idle.stl
- added link shoulder_right_frame; visual mesh filename=package://mh5_description/meshes/frame01.stl
Joints:
- added joint arm_left_fixed: type fixed, parent arm_left, child arm_left_fixed, origin xyz=0 -0.03675 0 rpy=0 1.5708 0
- added joint hip_left_fixed: type fixed, parent base_link, child hip_left, origin xyz=-0.0105 0.04575 -0.017 rpy=0 3.1416 1.5708
- added joint hip_right_fixed: type fixed, parent base_link, child hip_right, origin xyz=-0.0105 -0.04575 -0.017 rpy=0 3.1416 1.5708
- added joint l_elb_y: type revolute, parent arm_left_fixed, child elbow, origin xyz=0 -0.0213 0 rpy=0 0 1.5708, axis 1 0 0, limit lower=-3.1416 upper=3.1416 effort=1000 velocity=100
- added joint l_sho_p: type revolute, parent shoulder_left, child shoulder_left_frame, origin xyz=0 0 0.019 rpy=0 3.1416 0, axis 0 0 1, limit lower=-3.1416 upper=3.1416 effort=1000 velocity=100
- added joint l_sho_r: type revolute, parent shoulder_left_frame, child arm_left, origin xyz=0 -0.016 -0.027 rpy=0 1.5707 0, axis 0 0 1, limit lower=-3.1416 upper=3.1416 effort=1000 velocity=100
- added joint r_sho_p: type revolute, parent shoulder_right, child shoulder_right_frame, origin xyz=0 0 0.019 rpy=0 3.1416 3.1416, axis 0 0 -1, limit lower=-3.1416 upper=3.1416 effort=1000 velocity=100
- added joint shoulder_left_fixed: type fixed, parent base_link, child shoulder_left, origin xyz=-0.003 0.048 0.09175 rpy=1.5708 0 3.1416
- added joint shoulder_right_fixed: type fixed, parent base_link, child shoulder_right, origin xyz=-0.003 -0.048 0.09175 rpy=1.5708 0 0
