Commit message: reorg mh5_controller

File: mh5_description/urdf/mh5_robot_copy.xacro (robot description, xacro)
@@ -1,7 +1,4 @@
 <?xml version="1.0" ?>
 <robot xmlns:xacro="http://ros.org/wiki/xacro" name="mh5_robot">
-    <xacro:include filename="$(find mh5_description)/urdf/mh5_arm.xacro"/>
-    <xacro:include filename="$(find mh5_description)/urdf/mh5_leg.xacro"/>
-    <xacro:include filename="$(find mh5_description)/urdf/mh5_head.xacro"/>
     <xacro:macro name="material_ivory">
         <material name="ivory">
@@ -29,4 +26,9 @@
             </geometry>
         </collision>
+        <inertial>
+            <mass value="0.125444"/>
+            <inertia ixx="0.000328549" iyy="0.00043996" izz="0.000219472"
+                     ixy="0"           ixz="0"          iyz="0.000004439" />
+        </inertial>
     </link>
     <joint name="chest_fixed" type="fixed">
@@ -45,4 +47,15 @@
             </material>
         </visual>
+        <collision>
+            <origin rpy="${-pi/2} 0 ${-pi/2}" xyz="0 0 0"/>
+            <geometry>
+                <mesh filename="package://mh5_description/meshes/screen.stl"/>
+            </geometry>
+        </collision>
+        <inertial>
+            <mass value="0.0176"/>
+            <inertia ixx="0.000004545" iyy="0.000006293" izz="0.00000182"
+                     ixy="0"           ixz="0"          iyz="0" />
+        </inertial>
     </link>
     <joint name="screen_fixed" type="fixed">
@@ -51,8 +64,3 @@
         <origin xyz="0.02935 0 0.05426" rpy="0 0 0"/>
     </joint>
-    <xacro:mh5_head parent="chest"/>
-    <xacro:mh5_arm side="left" parent="chest"/>
-    <xacro:mh5_arm side="right" parent="chest"/>
-    <xacro:mh5_leg side="left" parent="chest"/>
-    <xacro:mh5_leg side="right" parent="chest"/>
 </robot>
