Commit message: finalisez urdf rev B

File: mh5_description/urdf/mh5_leg_revB.xacro (robot description, xacro)
@@ -151,5 +151,5 @@
             <parent link="${side}_tibia"/>
             <child link="${side}_ankle_servo"/>
-            <axis xyz="-1 0 0"/>
+            <axis xyz="1 0 0"/>
             <origin xyz="0 0 0" rpy="0 0 0"/>
             <limit lower="-${pi/2}" upper="${0.64*pi}" effort="${effort}" velocity="${velocity}"/>

File: mh5_description/urdf/mh5_robot_revB.xacro (robot description, xacro)
@@ -1,5 +1,5 @@
 <?xml version="1.0" ?>
 <robot xmlns:xacro="http://ros.org/wiki/xacro" name="mh5_robot">
-    <xacro:include filename="$(find mh5_description)/urdf/mh5_arm.xacro"/>
+    <xacro:include filename="$(find mh5_description)/urdf/mh5_arm_revB.xacro"/>
     <xacro:include filename="$(find mh5_description)/urdf/mh5_leg_revB.xacro"/>
     <xacro:include filename="$(find mh5_description)/urdf/mh5_head_revB.xacro"/>
@@ -48,4 +48,6 @@
     <xacro:mh5_leg side="left" parent="chest" />
     <xacro:mh5_leg side="right" parent="chest" />
+    <xacro:mh5_arm side="left" parent="chest" />
+    <xacro:mh5_arm side="right" parent="chest" />
     <gazebo>
         <plugin name="gazebo_ros_control" filename="libgazebo_ros_control.so">
