Commit message: fix arm urdf problem

File: mh5_description/urdf/mh5_arm_revB.xacro (robot description, xacro)
@@ -123,4 +123,21 @@
                 <material name="ivory"/>
             </visual>
+            <collision>
+                <origin rpy="0 0 0" xyz="0 0 0"/>
+                <geometry>
+                    <mesh filename="package://mh5_description/meshes/frame03_revB.stl"/>
+                </geometry>
+            </collision>
+            <inertial>
+                <origin rpy="0 0 0" xyz="0 0 0"/>
+                <mass value="0.0028"/>
+                <inertia
+                    ixx="0.000000349"
+                    iyy="0.000000241"
+                    izz="0.000000567"
+                    ixy="0"
+                    ixz="0"
+                    iyz="0" />
+            </inertial>
         </link>
         <joint name="${short_side}_elb_y" type="revolute">

File: mh5_description/urdf/mh5_robot_revB.xacro (robot description, xacro)
@@ -52,5 +52,4 @@
     <gazebo>
         <plugin name="gazebo_ros_control" filename="libgazebo_ros_control.so">
-            <robotNamespace>/</robotNamespace>
         </plugin>
         <plugin name="joint_state_publisher" filename="libgazebo_ros_joint_state_publisher.so">

File: mh5_description/urdf/mh5_transmission.xacro (robot description, xacro)
@@ -8,5 +8,4 @@
       </joint>
       <actuator name="${name}_motor">
-        <hardwareInterface>hardware_interface/PositionJointInterface</hardwareInterface>
         <mechanicalReduction>1</mechanicalReduction>
       </actuator>

Commit message: adjusted gazebo settings

File: mh5_description/urdf/mh5_arm_revB.xacro (robot description, xacro)
@@ -9,5 +9,5 @@
             <xacro:property name="factor" value = "-1.0"/>
         </xacro:if>
-        <xacro:property name="effort" value="1.5"/>
+        <xacro:property name="effort" value="1.0"/>
         <xacro:property name="velocity" value="${2*pi}"/>
         <joint name="${side}_shoulder_fixed" type="fixed">

File: mh5_description/urdf/mh5_head_revB.xacro (robot description, xacro)
@@ -8,5 +8,5 @@
             <child link="head_servo"/>
             <origin xyz="-0.007076 0 ${0.191046+0.019}" rpy="0 0 0"/>
-            <limit lower="-${pi/2}" upper="${pi/2}" effort="1000" velocity="100"/>
+            <limit lower="-${pi/2}" upper="${pi/2}" effort="1.0" velocity="${2*pi}"/>
         </joint>
         <xacro:insert_transmission name="head_y"/>
@@ -42,5 +42,5 @@
             <child link="head_frame"/>
             <origin xyz="-0.024 0 0" rpy="0 0 0"/>
-            <limit lower="-${pi/12}" upper="${pi/4}" effort="1000" velocity="100"/>
+            <limit lower="-${pi/12}" upper="${pi/4}" effort="1.0" velocity="${2*pi}"/>
         </joint>
         <xacro:insert_transmission name="head_p"/>

File: mh5_description/urdf/mh5_leg_revB.xacro (robot description, xacro)
@@ -10,6 +10,8 @@
             <xacro:property name="factor" value = "-1.0"/>
         </xacro:if>
-        <xacro:property name="effort" value="1.5"/>
+        <xacro:property name="effort" value="1000.0"/>
         <xacro:property name="velocity" value="${2*pi}"/>
+        <xacro:property name="damping" value="0.1"/>
+        <xacro:property name="friction" value="0.0"/>
         <joint name="${short_side}_hip_r" type="revolute">
             <parent link="${parent}"/>
@@ -18,4 +20,5 @@
             <origin xyz="0 ${factor*0.048} 0" rpy="0 0 0"/>
             <limit lower="-${pi/4}" upper="${3*pi/4}" effort="${effort}" velocity="${velocity}"/>
+            <dynamics damping="${damping}" friction="${friction}" />
         </joint>
         <xacro:insert_transmission name="${short_side}_hip_r"/>
@@ -52,4 +55,5 @@
             <origin xyz="0 0 -0.024" rpy="0 0 0"/>
             <limit lower="-${0.6*pi}" upper="${0.6*pi}" effort="${effort}" velocity="${velocity}"/>
+            <dynamics damping="${damping}" friction="${friction}" />
         </joint>
         <xacro:insert_transmission name="${short_side}_hip_p"/>
@@ -86,4 +90,5 @@
             <origin xyz="-0.024 0 -0.061" rpy="0 ${pi/2} 0"/>
             <limit lower="0" upper="${1.2*pi}" effort="${effort}" velocity="${velocity}"/>
+            <dynamics damping="${damping}" friction="${friction}" />
         </joint>
         <xacro:insert_transmission name="${short_side}_kne_p"/>
@@ -120,4 +125,5 @@
             <origin xyz="0.053 0 0.024" rpy="${pi/2} 0 -${pi/2}"/>
             <limit lower="-${pi/4}" upper="${pi/4}" effort="${effort}" velocity="${velocity}"/>
+            <dynamics damping="${damping}" friction="${friction}" />
         </joint>
         <xacro:insert_transmission name="${short_side}_kne_y"/>
@@ -154,4 +160,5 @@
             <origin xyz="0 0 0" rpy="0 0 0"/>
             <limit lower="-${pi/2}" upper="${0.64*pi}" effort="${effort}" velocity="${velocity}"/>
+            <dynamics damping="${damping}" friction="${friction}" />
         </joint>
         <xacro:insert_transmission name="${short_side}_ank_p"/>
@@ -188,4 +195,5 @@
             <origin xyz="0 0 -0.024" rpy="0 0 ${pi/2}"/>
             <limit lower="-${pi/2}" upper="${pi/2}" effort="${effort}" velocity="${velocity}"/>
+            <dynamics damping="${damping}" friction="${friction}" />
         </joint>
         <xacro:insert_transmission name="${short_side}_ank_r"/>
