Commit message: updated model for Gazebo

File: mh5_description/urdf/mh5_robot_revB.xacro (robot description, xacro)
@@ -43,5 +43,5 @@
         <parent link="base_link"/>
         <child link="chest"/>
-        <origin xyz="0 0 0.202" rpy="0 0 0"/>
+        <origin xyz="0 0 0.200" rpy="0 0 0"/>
     </joint>
     <xacro:mh5_head parent="chest" />
