Commit message: URDF leg rev C complete

File: mh5_description/urdf/mh5_leg_revC.xacro (robot description, xacro)
@@ -38,5 +38,4 @@
             </collision>
             <inertial>
-                <origin rpy="0 0 0" xyz="0 0 0"/>
                 <mass value="0.098"/>
                 <inertia
@@ -73,5 +72,4 @@
             </collision>
             <inertial>
-                <origin rpy="0 0 0" xyz="0 0 0"/>
                 <mass value="0.016"/>
                 <inertia
@@ -84,5 +82,5 @@
             </inertial>
         </link>
-        <!-- <joint name="${short_side}_kne_p" type="revolute">
+       <joint name="${short_side}_kne_p" type="revolute">
             <parent link="${side}_thigh"/>
             <child link="${side}_knee_servo"/>
@@ -95,26 +93,25 @@
         <link name="${side}_knee_servo">
             <visual>
-                <origin rpy="-${pi/2} 0 0" xyz="0 0 0.012"/>
-                <geometry>
-                    <mesh filename="package://mh5_description/meshes/2xl430_1_idle.stl"/>
+                <origin rpy="0 0 0" xyz="0 0 0.024"/>
+                <geometry>
+                    <mesh filename="package://mh5_description/meshes/2XL430_1_idle_revC.stl"/>
                 </geometry>
                 <xacro:material_black/>
             </visual>
             <collision>
-                <origin rpy="-${pi/2} 0 0" xyz="0 0 0.012"/>
-                <geometry>
-                    <mesh filename="package://mh5_description/meshes/2xl430_1_idle.stl"/>
-                </geometry>
-            </collision>
-            <inertial>
-                <origin rpy="-${pi/2} 0 0" xyz="0 0 0.012"/>
+                <origin rpy="0 0 0" xyz="0 0 0.024"/>
+                <geometry>
+                    <mesh filename="package://mh5_description/meshes/2XL430_1_idle_revC.stl"/>
+                </geometry>
+            </collision>
+            <inertial>
                 <mass value="0.098"/>
                 <inertia
                     ixx="0.000026983"
-                    iyy="0.000019139"
-                    izz="0.000026983"
-                    ixy="0"
-                    ixz="0.000000654"
-                    iyz="0.0" />
+                    iyy="0.000026983"
+                    izz="0.000019139"
+                    ixy="0.000000654"
+                    ixz="-0.000000001"
+                    iyz="0.000000002" />
             </inertial>
         </link>
@@ -123,5 +120,5 @@
             <child link="${side}_tibia"/>
             <axis xyz="0 0 ${factor}"/>
-            <origin xyz="0.053 0 0.024" rpy="${pi/2} 0 -${pi/2}"/>
+            <origin xyz="0.019 0 0.024" rpy="0 -${pi/2} 0"/>
             <limit lower="-${pi/4}" upper="${pi/4}" effort="${effort}" velocity="${velocity}"/>
             <dynamics damping="${damping}" friction="${friction}" />
@@ -132,5 +129,5 @@
                 <origin rpy="0 0 0" xyz="0 0 0"/>
                 <geometry>
-                    <mesh filename="package://mh5_description/meshes/frame02_revB.stl"/>
+                    <mesh filename="package://mh5_description/meshes/frame02_revC.stl"/>
                 </geometry>
                 <xacro:material_ivory/>
@@ -139,5 +136,5 @@
                 <origin rpy="0 0 0" xyz="0 0 0"/>
                 <geometry>
-                    <mesh filename="package://mh5_description/meshes/frame02_revB.stl"/>
+                    <mesh filename="package://mh5_description/meshes/frame02_revC.stl"/>
                 </geometry>
             </collision>
@@ -146,10 +143,10 @@
                 <mass value="0.0077"/>
                 <inertia
-                    ixx="0.000003238"
-                    iyy="0.000001387"
-                    izz="0.000002795"
-                    ixy="0"
-                    ixz="0"
-                    iyz="0" />
+                    ixx="0.000003217"
+                    iyy="0.000001377"
+                    izz="0.000002781"
+                    ixy="0.000000000"
+                    ixz="-0.000000011"
+                    iyz="0.000000000" />
             </inertial>
         </link>
@@ -158,5 +155,5 @@
             <child link="${side}_ankle_servo"/>
             <axis xyz="1 0 0"/>
-            <origin xyz="0 0 0" rpy="0 0 0"/>
+            <origin xyz="0 0 -0.034" rpy="0 0 -${pi/2}"/>
             <limit lower="-${pi/2}" upper="${0.64*pi}" effort="${effort}" velocity="${velocity}"/>
             <dynamics damping="${damping}" friction="${friction}" />
@@ -165,26 +162,25 @@
         <link name="${side}_ankle_servo">
             <visual>
-                <origin rpy="-${pi/2} 0 0" xyz="0 0 -0.012"/>
-                <geometry>
-                    <mesh filename="package://mh5_description/meshes/2xl430_2_idles.stl"/>
+                <origin rpy="0 0 0" xyz="0 0 0"/>
+                <geometry>
+                    <mesh filename="package://mh5_description/meshes/2XL430_2_idles_revC.stl"/>
                 </geometry>
                 <xacro:material_black/>
             </visual>
             <collision>
-                <origin rpy="-${pi/2} 0 0" xyz="0 0 -0.012"/>
-                <geometry>
-                    <mesh filename="package://mh5_description/meshes/2xl430_2_idles.stl"/>
-                </geometry>
-            </collision>
-            <inertial>
-                <origin rpy="-${pi/2} 0 0" xyz="0 0 -0.012"/>
+                <origin rpy="0 0 0" xyz="0 0 0"/>
+                <geometry>
+                    <mesh filename="package://mh5_description/meshes/2XL430_2_idles_revC.stl"/>
+                </geometry>
+            </collision>
+            <inertial>
                 <mass value="0.098"/>
                 <inertia
                     ixx="0.000026983"
-                    iyy="0.000019139"
-                    izz="0.000026983"
-                    ixy="0"
-                    ixz="0.000000654"
-                    iyz="0.0" />
+                    iyy="0.000026983"
+                    izz="0.000019139"
+                    ixy="0.000000654"
+                    ixz="-0.000000002"
+                    iyz="0.000000001" />
             </inertial>
         </link>
@@ -202,5 +198,5 @@
                 <origin rpy="0 0 0" xyz="0 0 0"/>
                 <geometry>
-                    <mesh filename="package://mh5_description/meshes/foot_${side}.stl"/>
+                    <mesh filename="package://mh5_description/meshes/foot_${side}_revC.stl"/>
                 </geometry>
                 <xacro:material_ivory/>
@@ -209,5 +205,5 @@
                 <origin rpy="0 0 0" xyz="0 0 0"/>
                 <geometry>
-                    <mesh filename="package://mh5_description/meshes/foot_${side}.stl"/>
+                    <mesh filename="package://mh5_description/meshes/foot_${side}_revC.stl"/>
                 </geometry>
             </collision>
@@ -216,10 +212,10 @@
                 <mass value="0.053"/>
                 <inertia
-                    ixx="0.000027287"
-                    iyy="0.000067414"
-                    izz="0.000083844"
-                    ixy="-0.000000277"
-                    ixz="0.000001204"
-                    iyz="0.0000000084" />
+                    ixx="0.000027639"
+                    iyy="0.000067044"
+                    izz="0.000083497"
+                    ixy="-0.000000056"
+                    ixz="0.000001332"
+                    iyz="0.0000000012" />
             </inertial>
         </link>
@@ -227,11 +223,11 @@
             <parent link="${side}_foot"/>
             <child link="${side}_battery"/>
-            <origin xyz="0 0 -0.037" rpy="0 0 0"/>
+            <origin xyz="0.003 0 -0.037" rpy="0 0 0"/>
         </joint>
         <link name="${side}_battery">
             <visual>
-                <origin rpy="0 0 -${pi/2}" xyz="0.003 0 0"/>
-                <geometry>
-                    <mesh filename="package://mh5_description/meshes/battery.stl"/>
+                <origin rpy="0 0 0" xyz="0 0 0"/>
+                <geometry>
+                    <mesh filename="package://mh5_description/meshes/battery_revC.stl"/>
                 </geometry>
                 <material name="blue">
@@ -240,21 +236,21 @@
             </visual>
             <collision>
-                <origin rpy="0 0 -${pi/2}" xyz="0 0 0"/>
-                <geometry>
-                    <mesh filename="package://mh5_description/meshes/battery.stl"/>
-                </geometry>
-            </collision>
-            <inertial>
-                <origin rpy="0 0 -${pi/2}" xyz="0 0 0"/>
+                <origin rpy="0 0 0" xyz="0 0 0"/>
+                <geometry>
+                    <mesh filename="package://mh5_description/meshes/battery_revC.stl"/>
+                </geometry>
+            </collision>
+            <inertial>
+                <origin rpy="0 0 0" xyz="0 0 0"/>
                 <mass value="0.155"/>
                 <inertia
-                    ixx="0.000144254"
-                    iyy="0.000034376"
+                    ixx="0.000034376"
+                    iyy="0.000144254"
                     izz="0.000173658"
-                    ixy="0"
-                    ixz="0"
-                    iyz="0" />
-            </inertial>
-        </link> -->
+                    ixy="0.000000000"
+                    ixz="0.000000000"
+                    iyz="0.000000000" />
+            </inertial>
+        </link>
     </xacro:macro>
 </robot>

File: mh5_description/urdf/mh5_robot_revC.xacro (robot description, xacro)
@@ -11,5 +11,5 @@
     <xacro:macro name="material_black">
         <material name="black">
-            <color rgba="0.1 0.1 0.1 1"/>
+            <color rgba="0.2 0.2 0.2 1"/>
         </material>
     </xacro:macro>
@@ -43,5 +43,5 @@
         <parent link="base_link"/>
         <child link="chest"/>
-        <origin xyz="0 0 0.200" rpy="0 0 0"/>
+        <origin xyz="0 0 0.203" rpy="0 0 0"/>
     </joint>
     <!-- <xacro:mh5_head parent="chest" /> -->
