Commit message: fix head direction in urdf

File: mh5_description/urdf/mh5_head_revC.xacro (robot description, xacro)
@@ -37,5 +37,5 @@
         </link>
         <joint name="head_p" type="revolute">
-            <axis xyz="0 -1 0"/>
+            <axis xyz="0 1 0"/>
             <parent link="head_servo"/>
             <child link="head_frame"/>

Commit message: fix head directions in urdf

File: mh5_description/urdf/mh5_head_revC.xacro (robot description, xacro)
@@ -4,5 +4,5 @@
     <xacro:macro name="mh5_head" params="parent">
         <joint name="head_y" type="revolute">
-            <axis xyz="1 0 0"/>
+            <axis xyz="-1 0 0"/>
             <parent link="${parent}"/>
             <child link="head_servo"/>
@@ -37,5 +37,5 @@
         </link>
         <joint name="head_p" type="revolute">
-            <axis xyz="0 1 0"/>
+            <axis xyz="0 -1 0"/>
             <parent link="head_servo"/>
             <child link="head_frame"/>
