Commit message: fix arm collision setting in URDF

File: mh5_description/urdf/mh5_arm_revC.xacro (robot description, xacro)
@@ -186,5 +186,5 @@
             </visual>
             <collision>
-                <origin rpy="0 0 0" xyz="0 0 0"/>
+                <origin rpy="0 0 0" xyz="0 0 -0.03925"/>
                 <geometry>
                     <mesh filename="package://mh5_description/meshes/lower_arm.stl"/>

Commit message: fix elb_p direction urdf

File: mh5_description/urdf/mh5_arm_revC.xacro (robot description, xacro)
@@ -203,5 +203,5 @@
         </link>
         <joint name="${short_side}_elb_p" type="revolute">
-            <axis xyz="${-factor} 0 0"/>
+            <axis xyz="${factor} 0 0"/>
             <parent link="${side}_lower_arm_frame"/>
             <child link="${side}_lower_arm_servo"/>
